File: 00_battery_safety.kicad_sch (KiCad schematic)
At the start: 32 parts, among them J15 LEFT MOTOR LARGE SOLDER PADS, J4 LEFT MOTOR + ENCODER, U2 VNH5019A-E

Commit message: Add whole-system battery cutoff and hardened servo interfaces
Parts:
- removed C12: 470 uF 35 V, Capacitor_THT:CP_Radial_D10.0mm_P5.00mm, symbol Device:C_Polarized
- removed C13: 100 nF 50 V, Capacitor_SMD:C_0805_2012Metric, symbol Device:C
- removed C14: 1 uF 25 V, Capacitor_SMD:C_0805_2012Metric, symbol Device:C
- removed C18: 100 nF 50 V FIT AT MOTOR - OFF BOARD, symbol Device:C
- removed C80: 10 nF current filter, Capacitor_SMD:C_0805_2012Metric, symbol Device:C
- removed D17: BAT54 LOW CLAMP, Diode_SMD:D_SOD-323, symbol Device:D_Schottky
- removed D18: BAT54 HIGH CLAMP, Diode_SMD:D_SOD-323, symbol Device:D_Schottky
- removed F5: 5 A MINI BLADE MOTOR BRANCH, Fuse:Fuseholder_Blade_Mini_Keystone_3568, symbol Device:Fuse
- removed F7: 100 mA PTC, Fuse:Fuse_0805_2012Metric, symbol Device:Polyfuse
- removed J15: LEFT MOTOR LARGE SOLDER PADS, Connector_Wire:SolderWire-1.5sqmm_1x02_P7.8mm_D1.7mm_OD3.9mm, symbol Connector_Generic:Conn_01x02
- removed J4: LEFT MOTOR + ENCODER, Connector_JST:JST_PH_B6B-PH-K_1x06_P2.00mm_Vertical, symbol Connector_Generic:Conn_01x06
- removed JP1, JP2: PH MOTOR POWER BYPASS - NORMALLY OPEN, Jumper:SolderJumper-2_P1.3mm_Open_Pad1.0x1.5mm, symbol Jumper:SolderJumper_2_Open
- removed R7: 680 R current sense, Resistor_SMD:R_0805_2012Metric, symbol Device:R
- removed R80, R81, R82: 1 k series, Resistor_SMD:R_0805_2012Metric, symbol Device:R
- removed R83, R84, R85: 10 k pulldown, Resistor_SMD:R_0805_2012Metric, symbol Device:R
- removed R86: 10 k fault pullup, Resistor_SMD:R_0805_2012Metric, symbol Device:R
- removed R88: 4.7 k ADC protect, Resistor_SMD:R_0805_2012Metric, symbol Device:R
- removed TP20: VBAT, TestPoint:TestPoint_Pad_D1.5mm, symbol Connector:TestPoint
- removed TP21: PWM, TestPoint:TestPoint_Pad_D1.5mm, symbol Connector:TestPoint
- removed TP22: INA, TestPoint:TestPoint_Pad_D1.5mm, symbol Connector:TestPoint
- removed TP23: INB, TestPoint:TestPoint_Pad_D1.5mm, symbol Connector:TestPoint
- removed TP24: DIAG, TestPoint:TestPoint_Pad_D1.5mm, symbol Connector:TestPoint
- removed TP25: CS ADC, TestPoint:TestPoint_Pad_D1.5mm, symbol Connector:TestPoint
- removed TP26: ENC A, TestPoint:TestPoint_Pad_D1.5mm, symbol Connector:TestPoint
- removed TP27: ENC B, TestPoint:TestPoint_Pad_D1.5mm, symbol Connector:TestPoint
- removed TP28: GND, TestPoint:TestPoint_Pad_D1.5mm, symbol Connector:TestPoint
- removed U2: VNH5019A-E, PickleballRobot:VNH5019_MultiPowerSO30_ThermalVias, symbol Driver_Motor:VNH5019A-E
- added C1: 1000 uF 35 V, Capacitor_THT:CP_Radial_D12.5mm_P5.00mm, symbol Device:C_Polarized
- added C2: 1 uF 25 V, Capacitor_SMD:C_0805_2012Metric, symbol Device:C
- added C4: 100 nF, Capacitor_SMD:C_0805_2012Metric, symbol Device:C
- added D1: SMBJ15CA, Diode_SMD:D_SMB, symbol Device:D_TVS
- added D14: BAT54 HIGH CLAMP, Diode_SMD:D_SOD-323, symbol Device:D_Schottky
- added D2: BAT54 LOW CLAMP, Diode_SMD:D_SOD-323, symbol Device:D_Schottky
- added D21: SMBJ15CA ACT TVS, Diode_SMD:D_SMB, symbol Device:D_TVS
- added D22: RED BATTERY CUTOFF, LED_SMD:LED_0805_2012Metric, symbol Device:LED
- added F1: 15 A ATO BLADE, Fuse:Fuse_Blade_ATO_directSolder, symbol Device:Fuse
- added J1: AMASS XT60PW-M BATTERY INPUT, Connector_AMASS:AMASS_XT60PW-M_1x02_P7.20mm_Horizontal, symbol Connector_Generic:Conn_01x02
- added J18: EXTERNAL NC LATCHING E-STOP LOOP, TerminalBlock_Phoenix:TerminalBlock_Phoenix_MKDS-3-2-5.08_1x02_P5.08mm_Horizontal, symbol Connector_Generic:Conn_01x02
- added J21: E-STOP RELAY COIL SUPPLY, TerminalBlock_Phoenix:TerminalBlock_Phoenix_MKDS-1,5-2-5.08_1x02_P5.08mm_Horizontal, symbol Connector_Generic:Conn_01x02
- added Q5, Q6: IRLB4030PBF 100 V 4.5 mR, Package_TO_SOT_THT:TO-220-3_Vertical, symbol Transistor_FET:Q_NMOS_GDS
- added R1: 100 k 1%, Resistor_SMD:R_0805_2012Metric, symbol Device:R
- added R115: 5.49 M 1% UV TOP, Resistor_SMD:R_0805_2012Metric, symbol Device:R
- added R116: 90.9 k 1% UV-OV, Resistor_SMD:R_0805_2012Metric, symbol Device:R
- added R117: 210 k 1% OV BOTTOM, Resistor_SMD:R_0805_2012Metric, symbol Device:R
- added R118: 100 k SHDN LIMIT, Resistor_SMD:R_0805_2012Metric, symbol Device:R
- added R119: 3.9 k LVD FAULT LED, Resistor_SMD:R_0805_2012Metric, symbol Device:R
- added R121, R122: 10 R GATE STOP, Resistor_SMD:R_0805_2012Metric, symbol Device:R
- added R2: 27 k 1%, Resistor_SMD:R_0805_2012Metric, symbol Device:R
- added R3: 1 k, Resistor_SMD:R_0805_2012Metric, symbol Device:R
- added TP64: BAT_RAW, TestPoint:TestPoint_Pad_D1.5mm, symbol Connector:TestPoint
- added TP65: BAT_FUSED, TestPoint:TestPoint_Pad_D1.5mm, symbol Connector:TestPoint
- added TP66: VBAT_SW, TestPoint:TestPoint_Pad_D1.5mm, symbol Connector:TestPoint
- added TP67: ACT_VBAT, TestPoint:TestPoint_Pad_D1.5mm, symbol Connector:TestPoint
- added TP68: GND, TestPoint:TestPoint_Pad_D1.5mm, symbol Connector:TestPoint
- added U12: LTC4365ITS8#TRPBF WHOLE-BOARD LVD, Package_TO_SOT_SMD:TSOT-23-8_HandSoldering, symbol Power_Management:LTC4365TS8
Connections:
- net 3V3: now also D14.1 (K)
- net ACT_VBAT: now also D21.1 (A1), J18.2 (Pin_2), TP67.1
- net GND: now also C1.2, C2.2, C4.2, D1.2 (A2), D2.2 (A), D21.2 (A2), J1.1 (Pin_1), J21.2 (Pin_2), R117.2, R2.2, TP68.1, U12.4 (GND)
- new net BAT_FUSED: F1.2, Q5.2 (D), R115.1, R118.1, R119.1, TP65.1, U12.1 (Vin)
- new net BAT_RAW: F1.1, J1.2 (Pin_2), TP64.1
- new net BAT_SENSE_RAW: R1.2, R2.1, R3.1
- new net GPIO33_BAT_ADC: C4.1, D14.2 (A), D2.1 (K), R3.2
- new net LVD_COMMON_SOURCE: Q5.3 (S), Q6.3 (S)
- new net LVD_FAULT: D22.1 (K), U12.6 (~{FAULT})
- new net LVD_GATE_DRV: R121.1, R122.1, U12.8 (GATE)
- new net LVD_GATE_Q5: Q5.1 (G), R121.2
- new net LVD_GATE_Q6: Q6.1 (G), R122.2
- new net LVD_LED_A: D22.2 (A), R119.2
- new net LVD_OV: R116.2, R117.1, U12.3 (OV)
- new net LVD_SHDN: R118.2, U12.5 (~{SHDN})
- new net LVD_UV: R115.2, R116.1, U12.2 (UV)
- new net VBAT_SW: C1.1, C2.1, D1.1 (A1), J18.1 (Pin_1), J21.1 (Pin_1), Q6.2 (D), R1.1, TP66.1, U12.7 (Vout)
- no-connect marks 1 -> 0
Other:
- note added: "3S BATTERY INPUT, FUSE, AND WHOLE-SYSTEM UV/OV DISCONNECT"
- note added: "ACTUATOR E-STOP LOOP"
- note added: "BATTERY VOLTAGE MONITOR"
- note added: "J21.1 -> XB5AS8442 NC button -> Panasonic CB1aF-RM-12V-A-5 coil -> J21.2. Relay NO contacts connect J18.1 to J18.2."
- note added: "LTC4365: about 9.6 V cutoff, 10.1 V reconnect, 13.8 V OV. This is a discharge cutoff, not a balance charger."
- note added: "The selected relay has internal coil suppression and a 40 A/14 VDC NO contact; pressing E-stop de-energizes it."
- note removed: "J15: primary red/white motor power. JP1/JP2 stay OPEN; bridge only for low-current JST-PH bench use."
- note removed: "J4/J5 cable: 1 RED motor+; 2 BLACK encoder GND; 3 YELLOW encoder A; 4 GREEN encoder B; 5 BLUE encoder +3V3; 6 WHITE motor-."
- note removed: "LEFT WHEEL MOTOR DRIVER"
- title: Left Wheel Motor Driver -> Battery Fuse, Whole-System Cutoff, and E-Stop
