File: 02_esp32_and_pi.kicad_sch (KiCad schematic)
At the start: 13 parts, among them J10 PI UART / CONTROL, J2 ESP32-PICO-KIT V4.1

Commit message: Complete pre-PCB electrical and safety audit
Parts:
- added D15, D16: 1N4148, Diode_SMD:D_SOD-323, symbol Device:D
- added J20: ACTUATOR ENABLE OVERRIDE DNP, Connector_PinHeader_2.54mm:PinHeader_1x02_P2.54mm_Vertical, symbol Connector_Generic:Conn_01x02
- added R43, R44: 0 R DNP, Resistor_SMD:R_0805_2012Metric, symbol Device:R
- added R45: 10 k, Resistor_SMD:R_0805_2012Metric, symbol Device:R
- added TP10: ACTUATOR_ENABLE, TestPoint:TestPoint_Loop_D2.50mm_Drill1.0mm, symbol Connector:TestPoint
- added TP11: MOTOR_DIAG, TestPoint:TestPoint_Loop_D2.50mm_Drill1.0mm, symbol Connector:TestPoint
- added TP12: GND, TestPoint:TestPoint_Loop_D2.50mm_Drill1.0mm, symbol Connector:TestPoint
- added TP7: 3V3, TestPoint:TestPoint_Loop_D2.50mm_Drill1.0mm, symbol Connector:TestPoint
- added TP8: PI_TX_TO_ESP, TestPoint:TestPoint_Loop_D2.50mm_Drill1.0mm, symbol Connector:TestPoint
- added TP9: ESP_TX_TO_PI, TestPoint:TestPoint_Loop_D2.50mm_Drill1.0mm, symbol Connector:TestPoint
- R42: value 10 k -> 100 k DEFAULT OFF
Connections:
- net 3V3: now also J20.1 (Pin_1), R45.2, TP7.1; no longer R42.2
- net ESP_TX_TO_PI: now also TP9.1
- net GND: now also J10.1 (Pin_1), R42.2, TP12.1
- net GPIO13_R_INA: now also J2.20 (Pin_20); no longer J2.18 (Pin_18)
- net GPIO21_I2C_SDA: now also R43.2; no longer J10.7 (Pin_7)
- net GPIO22_I2C_SCL: now also R44.2; no longer J10.8 (Pin_8)
- net MOTOR_DIAG: now also D15.1 (K), D16.1 (K), R45.1, TP11.1
- net PI_TX_TO_ESP: now also TP8.1
- net GPIO32_SERVO_OE: now reaches J2.10 (Pin_10)
- net GPIO5_RIGHT_DIAG: now reaches J2.11 (Pin_11)
- net GPIO19_PI_TX: now reaches J2.5 (Pin_5)
- net GPIO19_PI_TX: now also R41.1
- net GPIO23_LEFT_DIAG: now reaches J2.7 (Pin_7)
- net GPIO18_PI_RX: now reaches J2.9 (Pin_9)
- net GPIO18_PI_RX: now also R40.2
- net ESP_RX0_GPIO3: no longer names the net of J2.17 (Pin_17)
- net ESP_RX0_GPIO3: no longer R40.2
- net ESP_TX0_GPIO1: no longer names the net of J2.19 (Pin_19)
- net ESP_TX0_GPIO1: no longer R41.1
- net GPIO2_SERVO_OE: no longer names the net of J2.24 (Pin_24)
- net PI_ENABLE renamed ACTUATOR_ENABLE
- net ACTUATOR_ENABLE: now also J20.2 (Pin_2), TP10.1
- new net LEFT_DIAG: D15.2 (A)
- new net PI_I2C_SCL: J10.8 (Pin_8), R44.1
- new net PI_I2C_SDA: J10.7 (Pin_7), R43.1
- new net RIGHT_DIAG: D16.2 (A)
- no-connect marks 12 -> 9
Other:
- note added: "J10: 1/2 GND; 3 Pi TX->ESP GPIO18; 4 ESP GPIO19->Pi RX; 5 actuator enable; 6 fault; 7/8 I2C DNP."
- note added: "Pi: GPIO14 pin 8 -> J10.3; GPIO15 pin 10 <- J10.4; GPIO17 pin 11 -> J10.5; GND -> J10.1/2."
- note removed: "J10 pin 1 UNUSED; pin 2 GND; pin 3 Pi TX; pin 4 Pi RX; pins 5–8 optional control/I2C."
- note removed: "Pi GPIO14 physical pin 8 → J10.3; Pi GPIO15 physical pin 10 ← J10.4; Pi GND → J10.2."

Commit message: Correct critical controller schematic safety issues
Parts:
- removed D15, D16: 1N4148, Diode_SMD:D_SOD-323, symbol Device:D
- added D15, D16: BAT54 FAULT OR, Diode_SMD:D_SOD-323, symbol Device:D_Schottky
- added R46: 4.7 k OVERRIDE ISOLATION, Resistor_SMD:R_0805_2012Metric, symbol Device:R
- added R47: 1 k ESP FAULT SERIES, Resistor_SMD:R_0805_2012Metric, symbol Device:R
- J20: value ACTUATOR ENABLE OVERRIDE DNP -> SERVO ENABLE OVERRIDE DNP; now not fitted
- R42: value 100 k DEFAULT OFF -> 10 k DEFAULT OFF
- R43, R44: now not fitted
- TP10: value ACTUATOR_ENABLE -> SERVO_POWER_ENABLE; footprint TestPoint:TestPoint_Loop_D2.50mm_Drill1.0mm -> TestPoint:TestPoint_Pad_D1.5mm; now left out of the parts list
- TP11, TP12, TP7, TP8, TP9: footprint TestPoint:TestPoint_Loop_D2.50mm_Drill1.0mm -> TestPoint:TestPoint_Pad_D1.5mm; now left out of the parts list
Connections:
- net GND: now also D5.1 (K), D6.1 (K), D7.1 (K); no longer D5.2 (A), D6.2 (A), D7.2 (A)
- net LED_CTRL: now also D5.2 (A); no longer D5.1 (K)
- net LED_FAULT: now also D8.2 (A); no longer D8.1 (K)
- net LED_PI: now also D6.2 (A); no longer D6.1 (K)
- net LED_SERVO: now also D7.2 (A); no longer D7.1 (K)
- net LEFT_DIAG: now also D15.1 (K)
- net MOTOR_DIAG: now also D8.1 (K), D15.2 (A), D16.2 (A), R47.1; no longer D8.2 (A)
- net RIGHT_DIAG: now also D16.1 (K)
- net ACTUATOR_ENABLE renamed SERVO_POWER_ENABLE
- net SERVO_POWER_ENABLE: now also R46.2; no longer J20.2 (Pin_2)
- net GPIO23_LEFT_DIAG renamed GPIO23_MOTOR_DIAG
- net GPIO23_MOTOR_DIAG: now also R47.2
- net GPIO5_RIGHT_DIAG: no longer names the net of J2.11 (Pin_11)
- new net SERVO_ENABLE_OVERRIDE: J20.2 (Pin_2), R46.1
- no-connect marks 9 -> 10
Other:
- note added: "J10: 1/2 GND; 3 Pi TX->ESP GPIO18; 4 ESP GPIO19->Pi RX; 5 servo-power enable; 6 motor fault; 7/8 I2C DNP."
- note added: "Pi: GPIO14 pin8 -> J10.3; GPIO15 pin10 <- J10.4; GPIO17 pin11 -> J10.5; GPIO27 pin13 <- J10.6; GND -> J10.1/2."
- note removed: "J10: 1/2 GND; 3 Pi TX->ESP GPIO18; 4 ESP GPIO19->Pi RX; 5 actuator enable; 6 fault; 7/8 I2C DNP."
- note removed: "Pi: GPIO14 pin 8 -> J10.3; GPIO15 pin 10 <- J10.4; GPIO17 pin 11 -> J10.5; GND -> J10.1/2."
