File: 05_encoder_inputs.kicad_sch (KiCad schematic)
At the start: 12 parts, among them U6 74LVC1G14, U7 74LVC1G14, U8 74LVC1G14, U9 74LVC1G14

Commit message: Complete pre-PCB electrical and safety audit
Parts:
- added C84: 10 uF 10 V, Capacitor_SMD:C_0805_2012Metric, symbol Device:C
- added C85: 100 nF, Capacitor_SMD:C_0805_2012Metric, symbol Device:C
- added C86, C87, C88, C89: 100 nF local bypass, Capacitor_SMD:C_0805_2012Metric, symbol Device:C
- added FB1: BLM21PG221SN1D 220R@100MHz, Inductor_SMD:L_0805_2012Metric, symbol Device:FerriteBead
- added R72, R73, R74, R75: 1 k cable protection, Resistor_SMD:R_0805_2012Metric, symbol Device:R
- added TP40: ENC 3V3, TestPoint:TestPoint_Loop_D2.50mm_Drill1.0mm, symbol Connector:TestPoint
- added TP41: L A RAW, TestPoint:TestPoint_Loop_D2.50mm_Drill1.0mm, symbol Connector:TestPoint
- added TP42: L A OUT, TestPoint:TestPoint_Loop_D2.50mm_Drill1.0mm, symbol Connector:TestPoint
- added TP43: L B RAW, TestPoint:TestPoint_Loop_D2.50mm_Drill1.0mm, symbol Connector:TestPoint
- added TP44: L B OUT, TestPoint:TestPoint_Loop_D2.50mm_Drill1.0mm, symbol Connector:TestPoint
- added TP45: R A RAW, TestPoint:TestPoint_Loop_D2.50mm_Drill1.0mm, symbol Connector:TestPoint
- added TP46: R A OUT, TestPoint:TestPoint_Loop_D2.50mm_Drill1.0mm, symbol Connector:TestPoint
- added TP47: R B RAW, TestPoint:TestPoint_Loop_D2.50mm_Drill1.0mm, symbol Connector:TestPoint
- added TP48: R B OUT, TestPoint:TestPoint_Loop_D2.50mm_Drill1.0mm, symbol Connector:TestPoint
- added TP49: GND, TestPoint:TestPoint_Loop_D2.50mm_Drill1.0mm, symbol Connector:TestPoint
Connections:
- net 3V3: now also C86.1, C87.1, C88.1, C89.1, FB1.1
- net GND: now also C84.2, C85.2, C86.2, C87.2, C88.2, C89.2, TP49.1
- net GPIO34_ENC_LA: now also TP42.1
- net GPIO35_ENC_LB: now also TP44.1
- net GPIO37_ENC_RA: now also TP46.1
- net GPIO38_ENC_RB: now also TP48.1
- net LEFT_ENC_A_RAW: now also R72.2, TP41.1
- net LEFT_ENC_B_RAW: now also R73.2, TP43.1
- net RIGHT_ENC_A_RAW: now also R74.2, TP45.1
- net RIGHT_ENC_B_RAW: now also R75.2, TP47.1
- new net ENC_3V3: C84.1, C85.1, FB1.2, TP40.1
- new net LEFT_ENC_A_CABLE: R72.1
- new net LEFT_ENC_B_CABLE: R73.1
- new net RIGHT_ENC_A_CABLE: R74.1
- new net RIGHT_ENC_B_CABLE: R75.1

Commit message: Correct critical controller schematic safety issues
Parts:
- TP40, TP41, TP42, TP43, TP44, TP45, TP46, TP47, TP48, TP49: footprint TestPoint:TestPoint_Loop_D2.50mm_Drill1.0mm -> TestPoint:TestPoint_Pad_D1.5mm; now left out of the parts list
